File: Hardware/PROIECT.brd (EAGLE design)
At the start: 170.2 x 111.2 mm, 103 parts, among them IC1 BD5229G-TR, IC4 XC6220A331MR-G, J1 FH34SRJ-24S-0.5SH_99_, J2 SAMACSYS_PARTS_USB4110-GF-A, J3 QWIIC_RIGHT_ANGLE, J4 112A-TAAR-R03_ATTEND, Q1 20V/4.2A/52mΩ/1.4W, Q2 20V/4.2A/52mΩ/1.4W, Q3 SI1308EDL-T1-GE3, U1 W25Q512JVEIQ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

Commit message: update files after issues
Parts:
- TP1, TP10, TP11, TP12, TP13, TP14, TP15, TP16, TP17, TP2, TP3, TP4, TP5, TP6, TP7, TP8, TP9: value TPTP20R -> (none)
Routing:
- net GND: track 758.2 -> 1356.3 mm, vias 17 -> 60
- net 3V3: track 465.1 -> 467.0 mm
- net MOSI: track 199.1 -> 200.9 mm, vias 7 -> 8
- net SS_SD: track 66.2 -> 67.6 mm, vias 0 -> 2
- net EPD_CS: track 98.2 -> 99.4 mm
- net MISO: track 116.0 -> 116.8 mm
